Commit message: working with new cl gripper

File: spot_arm_moveit_config/config/spot.ros2_control.xacro (robot description, xacro)
@@ -9,6 +9,5 @@
             </hardware>
             <joint name="arm_sh0">
-                <command_interface name="position">
-                </command_interface>
+                <command_interface name="position"/>
                 <state_interface name="position">
                   <param name="initial_value">${initial_positions['arm_sh0']}</param>
@@ -58,4 +57,18 @@
                 <state_interface name="velocity"/>
             </joint>
+            <joint name="left_finger_joint">
+                <command_interface name="position"/>
+                <state_interface name="position">
+                  <param name="initial_value">${initial_positions['left_finger_joint']}</param>
+                </state_interface>
+                <state_interface name="velocity"/>
+            </joint>
+            <joint name="right_finger_joint">
+                <command_interface name="position"/>
+                <state_interface name="position">
+                  <param name="initial_value">${initial_positions['right_finger_joint']}</param>
+                </state_interface>
+                <state_interface name="velocity"/>
+            </joint>
         </ros2_control>
     </xacro:macro>

File: spot_arm_moveit_config/config/spot.urdf.xacro (robot description, xacro)
@@ -3,5 +3,5 @@
     <xacro:arg name="initial_positions_file" default="initial_positions.yaml" />
     <!-- Import spot urdf file -->
-    <xacro:include filename="$(find spot_description)/urdf/spot.urdf.xacro" />
+    <xacro:include filename="$(find spot_description)/urdf/spot_control.urdf.xacro" />
     <!-- Import control_xacro -->
     <xacro:include filename="spot.ros2_control.xacro" />

File: spot_description/urdf/spot_control.urdf.xacro (robot description, xacro)
@@ -1,5 +1,5 @@
 <?xml version="1.0" ?>
     <robot name="spot" xmlns:xacro="http://www.ros.org/wiki/xacro">
-      <xacro:include filename="$(find spot_description)/urdf/spot_macro_control.xacro" />
+      <xacro:include filename="$(find spot_description)/urdf/spot_macro_control_t.xacro" />
       <!-- Parameters -->
       <xacro:arg name="arm" default="true" />

File: spot_description/urdf/spot_macro_control_t.xacro (robot description, xacro)
@@ -378,44 +378,10 @@
         <material>Gazebo/DarkGrey</material>
     </gazebo>
-        <!-- CL gripper -->
+        <!-- CL -->
         <link name="${tf_prefix}griper_base_link">
-            <visual>
-                <origin xyz="0.12 -0.05 -0.07" rpy="1.57 0 1.57" />
-                    <geometry>
-                        <mesh filename="file://$(find spot_description)/meshes/arm/visual/base_grip.stl" scale="1000 1000 1000"/>
-                    </geometry>
-                    <material name="arm_link_wr1">
-                        <color rgba="0.2 0.2 0.2 1" />
-                    </material>
-            </visual>
-            <collision>
-                <geometry>
-                    <mesh filename="file://$(find spot_description)/meshes/arm/collision/base_grip.stl" scale="1000 1000 1000"/>
-                </geometry>
-            </collision>
-            <inertial>
-            <origin rpy="0.006393076449033863 0.2928526604761865 -0.022814984050994802"
-                xyz="0.12516802549362183 0.00010137435310753062 -0.013997982256114483" />
-            <mass value="0.785" />
-            <inertia ixx="0.00076741362048185" ixy="0.0" ixz="0.0" iyy="0.0017628124054271809" iyz="0.0"
-                izz="0.0016818105865345951" />
-            </inertial>
-        </link>
-        <joint name="${tf_prefix}grip_base_joint" type="fixed">
-            <origin xyz="0.0 0.0 0.0" rpy="0 0 0" />
-            <axis xyz="1 0 0" />
-            <parent link="${tf_prefix}arm_link_wr0" />
-            <child link="${tf_prefix}griper_base_link" />
-            <limit effort="1000" velocity="1000.00" lower="-2.87979326579064354163"
-                upper="2.87979326579064354163" />
-        </joint>
-        <gazebo reference="${tf_prefix}griper_base_link">
-            <material>Gazebo/DarkGrey</material>
-        </gazebo>
-        <link name="${tf_prefix}left_finger_link">
-        <visual>
-        <origin xyz="0.118 0.0 -0.07" rpy="1.57 0 0" />
-        <geometry>
-          <mesh filename="file://$(find spot_description)/meshes/arm/visual/left_finger.stl" scale="1000 1000 1000"/>
+      <visual>
+        <origin xyz="0.12 -0.05 -0.07" rpy="1.57 0 1.57" />
+        <geometry>
+          <mesh filename="package://spot_description/meshes/arm/visual/base_grip.stl" scale="1000 1000 1000"/>
         </geometry>
         <material name="arm_link_wr1">
@@ -425,5 +391,5 @@
       <collision>
         <geometry>
-          <mesh filename="file://$(find spot_description)/meshes/arm/collision/left_finger.stl" scale="1000 1000 1000"/>
+          <mesh filename="package://spot_description/meshes/arm/collision/base_grip.stl" scale="1000 1000 1000"/>
         </geometry>
       </collision>
@@ -436,20 +402,20 @@
       </inertial>
     </link>
-        <joint name="left_finger_joint" type="prismatic">
+        <joint name="${tf_prefix}grip_base_joint" type="fixed">
             <origin xyz="0.0 0.0 0.0" rpy="0 0 0" />
-            <axis xyz="0 1 0" />
-            <parent link="${tf_prefix}griper_base_link" />
-            <child link="${tf_prefix}left_finger_link" />
-            <limit effort="1000" velocity="1000.00" lower="-0.03"
-                upper="0.0" />
-        </joint>
-        <gazebo reference="${tf_prefix}left_finger_link">
-            <material>Gazebo/DarkGrey</material>
+            <axis xyz="1 0 0" />
+            <parent link="${tf_prefix}arm_link_wr0" />
+            <child link="${tf_prefix}griper_base_link" />
+            <limit effort="1000" velocity="1000.00" lower="-2.87979326579064354163"
+                upper="2.87979326579064354163" />
+        </joint>
+        <gazebo reference="${tf_prefix}griper_base_link">
+            <material>Gazebo/White</material>
         </gazebo>
-        <link name="${tf_prefix}right_finger_link">
+        <link name="${tf_prefix}left_finger_link">
       <visual>
-        <origin xyz="0.118 0.02 -0.07" rpy="1.57 0 0" />
-        <geometry>
-          <mesh filename="file://$(find spot_description)/meshes/arm/visual/right_finger.stl" scale="1000 1000 1000"/>
+        <origin xyz="0.118 0.0 -0.07" rpy="1.57 0 0" />
+        <geometry>
+          <mesh filename="package://spot_description/meshes/arm/visual/left_finger.stl" scale="1000 1000 1000"/>
         </geometry>
         <material name="arm_link_wr1">
@@ -459,5 +425,5 @@
       <collision>
         <geometry>
-          <mesh filename="file://$(find spot_description)/meshes/arm/collision/right_finger.stl" scale="1000 1000 1000"/>
+          <mesh filename="package://spot_description/meshes/arm/collision/left_finger.stl" scale="1000 1000 1000"/>
         </geometry>
       </collision>
@@ -470,15 +436,49 @@
       </inertial>
     </link>
-        <joint name="right_finger_joint" type="prismatic">
+        <joint name="${tf_prefix}left_finger_joint" type="prismatic">
+            <origin xyz="0.0 0.0 0.0" rpy="0 0 0" />
+            <axis xyz="0 1 0" />
+            <parent link="${tf_prefix}griper_base_link" />
+            <child link="${tf_prefix}left_finger_link" />
+            <limit effort="1000" velocity="1000.00" lower="-0.03"
+                upper="0.0" />
+        </joint>
+        <gazebo reference="${tf_prefix}left_finger_link">
+            <material>Gazebo/White</material>
+        </gazebo>
+        <link name="${tf_prefix}right_finger_link">
+      <visual>
+        <origin xyz="0.118 0.02 -0.07" rpy="1.57 0 0" />
+        <geometry>
+          <mesh filename="package://spot_description/meshes/arm/visual/right_finger.stl" scale="1000 1000 1000"/>
+        </geometry>
+        <material name="arm_link_wr1">
+          <color rgba="0.2 0.2 0.2 1" />
+        </material>
+      </visual>
+      <collision>
+        <geometry>
+          <mesh filename="package://spot_description/meshes/arm/collision/right_finger.stl" scale="1000 1000 1000"/>
+        </geometry>
+      </collision>
+      <inertial>
+        <origin rpy="0.006393076449033863 0.2928526604761865 -0.022814984050994802"
+          xyz="0.12516802549362183 0.00010137435310753062 -0.013997982256114483" />
+        <mass value="0.785" />
+        <inertia ixx="0.00076741362048185" ixy="0.0" ixz="0.0" iyy="0.0017628124054271809" iyz="0.0"
+          izz="0.0016818105865345951" />
+      </inertial>
+    </link>
+        <joint name="${tf_prefix}right_finger_joint" type="prismatic">
             <origin xyz="0.0 0.0 0.0" rpy="0 0 0" />
             <axis xyz="0 1 0" />
             <parent link="${tf_prefix}griper_base_link" />
             <child link="${tf_prefix}right_finger_link" />
-            <!--mimic joint="left_finger_joint" multiplier="-1" offset="0" /-->
+            <!--mimic joint="${tf_prefix}left_finger_joint" multiplier="-1" offset="0" /-->
             <limit effort="1000" velocity="1000.00" lower="-0.0"
             upper="0.03" />
         </joint>
         <gazebo reference="${tf_prefix}right_finger_link">
-            <material>Gazebo/DarkGrey</material>
+            <material>Gazebo/White</material>
         </gazebo>
         <!-- Extrematies -->
@@ -828,271 +828,5 @@
         </joint>
         <!-- Control plugins-->
-        <ros2_control name="GazeboSystem" type="system">
-                <hardware>
-                    <plugin>gazebo_ros2_control/GazeboSystem</plugin>
-                </hardware>
-                <joint name="${tf_prefix}arm_sh0">
-                    <command_interface name="position">
-                    </command_interface>
-                    <state_interface name="position">
-                        <param name="initial_value">0.0</param>
-                    </state_interface>
-                    <state_interface name="velocity"/>
-                </joint>
-                <joint name="${tf_prefix}arm_sh1">
-                    <command_interface name="position">
-                    </command_interface>
-                    <state_interface name="position">
-                        <param name="initial_value">-3.12</param>
-                    </state_interface>
-                    <state_interface name="velocity"/>
-                </joint>
-                <joint name="${tf_prefix}arm_el0">
-                    <command_interface name="position">
-                    </command_interface>
-                    <state_interface name="position">
-                         <param name="initial_value">3.12</param>
-                    </state_interface>
-                    <state_interface name="velocity"/>
-                </joint>
-                <joint name="${tf_prefix}arm_el1">
-                    <command_interface name="position">
-                    </command_interface>
-                    <state_interface name="position">
-                        <param name="initial_value">0.0</param>
-                    </state_interface>
-                    <state_interface name="velocity"/>
-                </joint>
-                <joint name="${tf_prefix}arm_wr0">
-                    <command_interface name="position">
-                    </command_interface>
-                    <state_interface name="position">
-                        <param name="initial_value">0.0</param>
-                    </state_interface>
-                    <state_interface name="velocity"/>
-                </joint>
-                <joint name="${tf_prefix}arm_wr1">
-                    <command_interface name="position">
-                    </command_interface>
-                    <state_interface name="position">
-                        <param name="initial_value">0.0</param>
-                    </state_interface>
-                    <state_interface name="velocity"/>
-                </joint>
-                <joint name="${tf_prefix}arm_f1x">
-                    <command_interface name="position">
-                    </command_interface>
-                    <state_interface name="position">
-                        <param name="initial_value">0.0</param>
-                    </state_interface>
-                    <state_interface name="velocity"/>
-                </joint>
-                <joint name="left_finger_joint">
-                    <command_interface name="position">
-                    </command_interface>
-                    <state_interface name="position">
-                        <param name="initial_value">0.0</param>
-                    </state_interface>
-                    <state_interface name="velocity"/>
-                </joint>
-                <joint name="right_finger_joint">
-                    <command_interface name="position">
-                    </command_interface>
-                    <state_interface name="position">
-                        <param name="initial_value">0.0</param>
-                    </state_interface>
-                    <state_interface name="velocity"/>
-                </joint>
-     </ros2_control>
-        <gazebo>
-            <plugin filename="libgazebo_ros2_control.so" name="gazebo_ros2_control">
-                <robot_sim_type>gazebo_ros2_control/GazeboSystem</robot_sim_type>
-                <parameters>$(find spot_arm_moveit_config)/config/ros2_controllers.yaml </parameters>
-            </plugin>
-        </gazebo>
         <!-- Sensor plaugins-->
-        <link name="pointcloud_link">
-            <visual>
-                <geometry>
-                    <sphere radius="0.010"/>
-                </geometry>
-            </visual>
-        </link>
-        <joint name="pointcloud_link_joint" type="fixed">
-            <origin rpy="0 0 0" xyz="0.151 0.0 0.02"/>
-            <parent link="arm_link_wr1"/>
-            <child link="pointcloud_link"/>
-            <axis xyz="0 0 0"/>
-        </joint>
-        <gazebo reference="pointcloud_link">
-            <sensor type="ray" name="pointcloud_sensor">
-            <ray>
-                <scan>
-                    <horizontal>
-                        <samples>10</samples>
-                        <resolution>1</resolution>
-                        <min_angle>-0.014835</min_angle>
-                         <max_angle>0.014835</max_angle>
-                    </horizontal>
-                    <vertical>
-                        <samples>10</samples>
-                        <resolution>1</resolution>
-                        <min_angle>-0.014835</min_angle>
-                        <max_angle>0.014835</max_angle>
-                    </vertical>
-                </scan>
-                <range>
-                     <min>0.10</min>
-                    <max>5.0</max>
-                    <resolution>0.001</resolution>
-                </range>
-          <!-- Using gazebo's noise instead of plugin's -->
-                <noise>
-                    <type>gaussian</type>
-                    <mean>0.0</mean>
-                    <stddev>0.001</stddev>
-                </noise>
-            </ray>
-          <!-- Using gazebo's update rate instead of plugin's -->
-            <update_rate>30</update_rate>
-          <plugin name="gazebo_ros_block_laser_controller" filename="libgazebo_ros_ray_sensor.so">
-          <!-- Change namespace and output topic so published topic is /rrbot/laser/pointcloud -->
-              <ros>
-                <namespace>spot</namespace>
-                <argument>~/out:=pointcloud</argument>
-              </ros>
-              <!-- Set output to sensor_msgs/PointCloud to get same output type as gazebo_ros_block_laser -->
-              <output_type>sensor_msgs/PointCloud</output_type>
-              <frame_name>pointcloud_link</frame_name>
-              <!-- min_intensity instead of hokuyoMinIntensity -->
-              <min_intensity>100.0</min_intensity>
-          </plugin>
-      </sensor>
-  </gazebo>
-        <!-- RGB CAMERA -->
-        <link name="rgb_camera_link_frame">
-        </link>
-        <joint name="rgb_camera_link_frame_joint" type="fixed">
-            <origin rpy="0 0 0" xyz="0.051 0.0 0.05"/>
-            <parent link="arm_link_wr1" />
-            <child link="rgb_camera_link_frame" />
-            <axis xyz="0 0 0"/>
-        </joint>
-        <!--gazebo reference="rgb_camera_link_frame">
-            <sensor name="camera" type="wideanglecamera">
-            <camera>
-                <horizontal_fov>6.283</horizontal_fov>
-                    <image>
-                        <width>320</width>
-                        <height>240</height>
-                    </image>
-                    <clip>
-                        <near>0.1</near>
-                        <far>100</far>
-                    </clip>
-                    <lens>
-                        <type>custom</type>
-                        <custom_function>
-                            <c1>1.05</c1>
-                            <c2>4</c2>
-                            <f>1.0</f>
-                            <fun>tan</fun>
-                        </custom_function>
-                        <scale_to_hfov>true</scale_to_hfov>
-                        <cutoff_angle>3.1415</cutoff_angle>
-                        <env_texture_size>512</env_texture_size>
-                    </lens>
-                    <always_on>1</always_on>
-                    <update_rate>30</update_rate>
-            </camera>
-            <plugin name="camera_controller" filename="libgazebo_ros_camera.so">
-                <cameraName>rgb_camera</cameraName>
-                <imageTopicName>image_raw</imageTopicName>
-                <cameraInfoTopicName>camera_info</cameraInfoTopicName>
-                <frameName>rgb_camera_link_frame</frameName>
-                <hackBaseline>0.07</hackBaseline>
-            </plugin>
-            </sensor>
-    </gazebo-->
-        <!-- *********************** CAMERA SETUP *********************************  -->
-<!-- Each sensor must be attached to a link.                              -->
-        <joint name="camera_joint" type="fixed">
-            <parent link="arm_link_wr1"/>
-            <child link="camera_link"/>
-            <origin xyz="0.14 0.0 0.02" rpy="0 0 0"/>
-        </joint>
-        <link name="camera_link">
-            <visual>
-                <geometry>
-                    <box size="0.010 0.03 0.03"/>
-                </geometry>
-            </visual>
-        </link>
-        <joint name="camera_optical_joint" type="fixed">
-        <parent link="camera_link"/>
-        <child link="camera_link_optical"/>
-        <origin xyz="0 0 0" rpy="${-pi/2} 0 ${-pi/2}"/>
-    </joint>
-        <link name="camera_link_optical"></link>
-        <gazebo reference="camera_link">
-            <sensor name="camera" type="camera">
-                <pose> 0 0 0 0 0 0 </pose>
-                <visualize>false</visualize>
-                <update_rate>30</update_rate>
-                <camera>
-                    <horizontal_fov>1.089</horizontal_fov>
-                    <image>
-                        <format>R8G8B8</format>
-                        <width>640</width>
-                        <height>480</height>
-                    </image>
-                    <clip>
-                        <near>0.05</near>
-                        <far>8.0</far>
-                    </clip>
-                </camera>
-            <plugin name="camera_controller" filename="libgazebo_ros_camera.so">
-                <frame_name>camera_link_optical</frame_name>
-            </plugin>
-        </sensor>
-    </gazebo>
-        <!--gazebo reference="camera_link">
-            <sensor name="camera" type="camera">
-                <update_rate>30.0</update_rate>
-                <always_on>1</always_on>
-                <camera name="camera">
-                    <horizontal_fov>1.3962634</horizontal_fov>
-                    <image>
-                        <width>480</width>
-                        <height>360</height>
-                        <format>R8G8B8</format>
-                    </image>
-                    <clip>
-                        <near>0.01</near>
-                        <far>20</far>
-                    </clip>
-                    <distortion>
-                        <k1>0.0</k1>
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