Commit message: working new move_group split the gripper action to three move groups

File: spot_description/urdf/spot_macro.xacro (robot description, xacro)
@@ -378,4 +378,105 @@
         <material>Gazebo/DarkGrey</material>
     </gazebo>
+         <!-- CL gripper -->
+        <link name="${tf_prefix}griper_base_link">
+            <visual>
+                <origin xyz="0.12 -0.05 -0.07" rpy="1.57 0 1.57" />
+                    <geometry>
+                        <mesh filename="file://$(find spot_description)/meshes/arm/visual/base_grip.stl" scale="1000 1000 1000"/>
+                    </geometry>
+                    <material name="arm_link_wr1">
+                        <color rgba="0.2 0.2 0.2 1" />
+                    </material>
+            </visual>
+            <collision>
+                <geometry>
+                    <mesh filename="file://$(find spot_description)/meshes/arm/collision/base_grip.stl" scale="1000 1000 1000"/>
+                </geometry>
+            </collision>
+            <inertial>
+            <origin rpy="0.006393076449033863 0.2928526604761865 -0.022814984050994802"
+                xyz="0.12516802549362183 0.00010137435310753062 -0.013997982256114483" />
+            <mass value="0.785" />
+            <inertia ixx="0.00076741362048185" ixy="0.0" ixz="0.0" iyy="0.0017628124054271809" iyz="0.0"
+                izz="0.0016818105865345951" />
+            </inertial>
+        </link>
+        <joint name="${tf_prefix}grip_base_joint" type="fixed">
+            <origin xyz="0.0 0.0 0.0" rpy="0 0 0" />
+            <parent link="${tf_prefix}arm_link_wr1" />
+            <child link="${tf_prefix}griper_base_link" />
+            <limit effort="1000" velocity="1000.00" lower="-2.87979326579064354163"
+                upper="2.87979326579064354163" />
+        </joint>
+        <gazebo reference="${tf_prefix}griper_base_link">
+            <material>Gazebo/DarkGrey</material>
+        </gazebo>
+        <link name="${tf_prefix}left_finger_link">
+        <visual>
+        <origin xyz="0.118 0.0 -0.07" rpy="1.57 0 0" />
+        <geometry>
+          <mesh filename="file://$(find spot_description)/meshes/arm/visual/left_finger.stl" scale="1000 1000 1000"/>
+        </geometry>
+        <material name="arm_link_wr1">
+          <color rgba="0.2 0.2 0.2 1" />
+        </material>
+      </visual>
+      <collision>
+        <geometry>
+          <mesh filename="file://$(find spot_description)/meshes/arm/collision/left_finger.stl" scale="1000 1000 1000"/>
+        </geometry>
+      </collision>
+      <inertial>
+        <origin rpy="0.006393076449033863 0.2928526604761865 -0.022814984050994802"
+          xyz="0.12516802549362183 0.00010137435310753062 -0.013997982256114483" />
+        <mass value="0.785" />
+        <inertia ixx="0.00076741362048185" ixy="0.0" ixz="0.0" iyy="0.0017628124054271809" iyz="0.0"
+          izz="0.0016818105865345951" />
+      </inertial>
+    </link>
+        <joint name="left_finger_joint" type="prismatic">
+            <origin xyz="0.0 0.0 0.0" rpy="0 0 0" />
+            <axis xyz="0 1 0" />
+            <parent link="${tf_prefix}griper_base_link" />
+            <child link="${tf_prefix}left_finger_link" />
+            <limit effort="1000" velocity="1000.00" lower="-0.03"
+                upper="0.0" />
+        </joint>
+        <gazebo reference="${tf_prefix}left_finger_link">
+            <material>Gazebo/DarkGrey</material>
+        </gazebo>
+        <link name="${tf_prefix}right_finger_link">
+      <visual>
+        <origin xyz="0.118 0.02 -0.07" rpy="1.57 0 0" />
+        <geometry>
+          <mesh filename="file://$(find spot_description)/meshes/arm/visual/right_finger.stl" scale="1000 1000 1000"/>
+        </geometry>
+        <material name="arm_link_wr1">
+          <color rgba="0.2 0.2 0.2 1" />
+        </material>
+      </visual>
+      <collision>
+        <geometry>
+          <mesh filename="file://$(find spot_description)/meshes/arm/collision/right_finger.stl" scale="1000 1000 1000"/>
+        </geometry>
+      </collision>
+      <inertial>
+        <origin rpy="0.006393076449033863 0.2928526604761865 -0.022814984050994802"
+          xyz="0.12516802549362183 0.00010137435310753062 -0.013997982256114483" />
+        <mass value="0.785" />
+        <inertia ixx="0.00076741362048185" ixy="0.0" ixz="0.0" iyy="0.0017628124054271809" iyz="0.0"
+          izz="0.0016818105865345951" />
+      </inertial>
+    </link>
+        <joint name="right_finger_joint" type="prismatic">
+            <origin xyz="0.0 0.0 0.0" rpy="0 0 0" />
+            <axis xyz="0 1 0" />
+            <parent link="${tf_prefix}griper_base_link" />
+            <child link="${tf_prefix}right_finger_link" />
+            <limit effort="1000" velocity="1000.00" lower="-0.0" upper="0.03" />
+        </joint>
+        <gazebo reference="${tf_prefix}right_finger_link">
+            <material>Gazebo/DarkGrey</material>
+        </gazebo>
         <!-- Extrematies -->
         <link name="${tf_prefix}front_left_hip">

File: spot_description/urdf/spot_macro_control.xacro (robot description, xacro)
@@ -378,4 +378,106 @@
         <material>Gazebo/DarkGrey</material>
     </gazebo>
+         <!-- CL gripper -->
+        <link name="${tf_prefix}griper_base_link">
+            <visual>
+                <origin xyz="0.12 -0.05 -0.07" rpy="1.57 0 1.57" />
+                    <geometry>
+                        <mesh filename="file://$(find spot_description)/meshes/arm/visual/base_grip.stl" scale="1000 1000 1000"/>
+                    </geometry>
+                    <material name="arm_link_wr1">
+                        <color rgba="0.2 0.2 0.2 1" />
+                    </material>
+            </visual>
+            <collision>
+                <geometry>
+                    <mesh filename="file://$(find spot_description)/meshes/arm/collision/base_grip.stl" scale="1000 1000 1000"/>
+                </geometry>
+            </collision>
+            <inertial>
+            <origin rpy="0.006393076449033863 0.2928526604761865 -0.022814984050994802"
+                xyz="0.12516802549362183 0.00010137435310753062 -0.013997982256114483" />
+            <mass value="0.785" />
+            <inertia ixx="0.00076741362048185" ixy="0.0" ixz="0.0" iyy="0.0017628124054271809" iyz="0.0"
+                izz="0.0016818105865345951" />
+            </inertial>
+        </link>
+        <joint name="${tf_prefix}grip_base_joint" type="fixed">
+            <origin xyz="0.0 0.0 0.0" rpy="0 0 0" />
+            <axis xyz="1 0 0" />
+            <parent link="${tf_prefix}arm_link_wr1" />
+            <child link="${tf_prefix}griper_base_link" />
+            <limit effort="1000" velocity="1000.00" lower="-2.87979326579064354163"
+                upper="2.87979326579064354163" />
+        </joint>
+        <gazebo reference="${tf_prefix}griper_base_link">
+            <material>Gazebo/DarkGrey</material>
+        </gazebo>
+        <link name="${tf_prefix}left_finger_link">
+        <visual>
+        <origin xyz="0.118 0.0 -0.07" rpy="1.57 0 0" />
+        <geometry>
+          <mesh filename="file://$(find spot_description)/meshes/arm/visual/left_finger.stl" scale="1000 1000 1000"/>
+        </geometry>
+        <material name="arm_link_wr1">
+          <color rgba="0.2 0.2 0.2 1" />
+        </material>
+      </visual>
+      <collision>
+        <geometry>
+          <mesh filename="file://$(find spot_description)/meshes/arm/collision/left_finger.stl" scale="1000 1000 1000"/>
+        </geometry>
+      </collision>
+      <inertial>
+        <origin rpy="0.006393076449033863 0.2928526604761865 -0.022814984050994802"
+          xyz="0.12516802549362183 0.00010137435310753062 -0.013997982256114483" />
+        <mass value="0.785" />
+        <inertia ixx="0.00076741362048185" ixy="0.0" ixz="0.0" iyy="0.0017628124054271809" iyz="0.0"
+          izz="0.0016818105865345951" />
+      </inertial>
+    </link>
+        <joint name="left_finger_joint" type="prismatic">
+            <origin xyz="0.0 0.0 0.0" rpy="0 0 0" />
+            <axis xyz="0 1 0" />
+            <parent link="${tf_prefix}griper_base_link" />
+            <child link="${tf_prefix}left_finger_link" />
+            <limit effort="1000" velocity="1000.00" lower="-0.03"
+                upper="0.0" />
+        </joint>
+        <gazebo reference="${tf_prefix}left_finger_link">
+            <material>Gazebo/DarkGrey</material>
+        </gazebo>
+        <link name="${tf_prefix}right_finger_link">
+      <visual>
+        <origin xyz="0.118 0.02 -0.07" rpy="1.57 0 0" />
+        <geometry>
+          <mesh filename="file://$(find spot_description)/meshes/arm/visual/right_finger.stl" scale="1000 1000 1000"/>
+        </geometry>
+        <material name="arm_link_wr1">
+          <color rgba="0.2 0.2 0.2 1" />
+        </material>
+      </visual>
+      <collision>
+        <geometry>
+          <mesh filename="file://$(find spot_description)/meshes/arm/collision/right_finger.stl" scale="1000 1000 1000"/>
+        </geometry>
+      </collision>
+      <inertial>
+        <origin rpy="0.006393076449033863 0.2928526604761865 -0.022814984050994802"
+          xyz="0.12516802549362183 0.00010137435310753062 -0.013997982256114483" />
+        <mass value="0.785" />
+        <inertia ixx="0.00076741362048185" ixy="0.0" ixz="0.0" iyy="0.0017628124054271809" iyz="0.0"
+          izz="0.0016818105865345951" />
+      </inertial>
+    </link>
+        <joint name="right_finger_joint" type="prismatic">
+            <origin xyz="0.0 0.0 0.0" rpy="0 0 0" />
+            <axis xyz="0 1 0" />
+            <parent link="${tf_prefix}griper_base_link" />
+            <child link="${tf_prefix}right_finger_link" />
+            <limit effort="1000" velocity="1000.00" lower="-0.0" upper="0.03" />
+        </joint>
+        <gazebo reference="${tf_prefix}right_finger_link">
+            <material>Gazebo/DarkGrey</material>
+        </gazebo>
         <!-- Extrematies -->
         <link name="${tf_prefix}front_left_hip">
@@ -784,9 +886,25 @@
                     <state_interface name="velocity"/>
                 </joint>
+                <joint name="left_finger_joint">
+                    <command_interface name="position">
+                    </command_interface>
+                    <state_interface name="position">
+                        <param name="initial_value">0.0</param>
+                    </state_interface>
+                    <state_interface name="velocity"/>
+                </joint>
+                <joint name="right_finger_joint">
+                    <command_interface name="position">
+                    </command_interface>
+                    <state_interface name="position">
+                        <param name="initial_value">0.0</param>
+                    </state_interface>
+                    <state_interface name="velocity"/>
+                </joint>
      </ros2_control>
         <gazebo>
             <plugin filename="libgazebo_ros2_control.so" name="gazebo_ros2_control">
                 <robot_sim_type>gazebo_ros2_control/GazeboSystem</robot_sim_type>
-                <parameters>$(find spot_arm_gazebo)/config/ros2_controllers.yaml </parameters>
+                <parameters>$(find arm_moveit_config)/config/ros2_controllers.yaml </parameters>
             </plugin>
         </gazebo>
