Commit message: Rebuild the arm_moveit_config package with additional set positions

File: spot_description/urdf/spot_macro_control.xacro (robot description, xacro)
@@ -424,4 +424,5 @@
       </visual>
       <collision>
+          <origin xyz="0.118 0.0 -0.07" rpy="1.57 0 0" />
         <geometry>
           <mesh filename="file://$(find spot_description)/meshes/arm/collision/left_finger.stl" scale="1000 1000 1000"/>
@@ -458,4 +459,5 @@
       </visual>
       <collision>
+          <origin xyz="0.118 0.02 -0.07" rpy="1.57 0 0" />
         <geometry>
           <mesh filename="file://$(find spot_description)/meshes/arm/collision/right_finger.stl" scale="1000 1000 1000"/>

Commit message: Modified gripper stl files

File: spot_description/urdf/spot_macro_control.xacro (robot description, xacro)
@@ -417,5 +417,5 @@
         <origin xyz="0.118 0.0 -0.07" rpy="1.57 0 0" />
         <geometry>
-          <mesh filename="file://$(find spot_description)/meshes/arm/visual/left_finger.stl" scale="1000 1000 1000"/>
+          <mesh filename="file://$(find spot_description)/meshes/arm/visual/left_finger_2.stl" scale="1000 1000 1000"/>
         </geometry>
         <material name="arm_link_wr1">
@@ -426,5 +426,5 @@
           <origin xyz="0.118 0.0 -0.07" rpy="1.57 0 0" />
         <geometry>
-          <mesh filename="file://$(find spot_description)/meshes/arm/collision/left_finger.stl" scale="1000 1000 1000"/>
+          <mesh filename="file://$(find spot_description)/meshes/arm/collision/left_finger_2.stl" scale="1000 1000 1000"/>
         </geometry>
       </collision>
@@ -442,5 +442,5 @@
             <parent link="${tf_prefix}griper_base_link" />
             <child link="${tf_prefix}left_finger_link" />
-            <limit effort="1000" velocity="1000.00" lower="-0.03"
+            <limit effort="1" velocity="10.00" lower="-0.03"
                 upper="0.0" />
         </joint>
@@ -452,5 +452,5 @@
         <origin xyz="0.118 0.02 -0.07" rpy="1.57 0 0" />
         <geometry>
-          <mesh filename="file://$(find spot_description)/meshes/arm/visual/right_finger.stl" scale="1000 1000 1000"/>
+          <mesh filename="file://$(find spot_description)/meshes/arm/visual/right_finger_2.stl" scale="1000 1000 1000"/>
         </geometry>
         <material name="arm_link_wr1">
@@ -461,5 +461,5 @@
           <origin xyz="0.118 0.02 -0.07" rpy="1.57 0 0" />
         <geometry>
-          <mesh filename="file://$(find spot_description)/meshes/arm/collision/right_finger.stl" scale="1000 1000 1000"/>
+          <mesh filename="file://$(find spot_description)/meshes/arm/collision/right_finger_2.stl" scale="1000 1000 1000"/>
         </geometry>
       </collision>
@@ -477,5 +477,5 @@
             <parent link="${tf_prefix}griper_base_link" />
             <child link="${tf_prefix}right_finger_link" />
-            <limit effort="1000" velocity="1000.00" lower="-0.0" upper="0.03" />
+            <limit effort="1" velocity="10.00" lower="-0.0" upper="0.03" />
         </joint>
         <gazebo reference="${tf_prefix}right_finger_link">
@@ -1044,6 +1044,6 @@
                     <image>
                         <format>R8G8B8</format>
-                        <width>640</width>
-                        <height>480</height>
+                        <width>1920</width>
+                        <height>1080</height>
                     </image>
                     <clip>

Commit message: Modified gripper stl files

File: spot_description/urdf/spot_macro_control.xacro (robot description, xacro)
@@ -417,5 +417,5 @@
         <origin xyz="0.118 0.0 -0.07" rpy="1.57 0 0" />
         <geometry>
-          <mesh filename="file://$(find spot_description)/meshes/arm/visual/left_finger_2.stl" scale="1000 1000 1000"/>
+          <mesh filename="file://$(find spot_description)/meshes/arm/visual/left_finger.stl" scale="1000 1000 1000"/>
         </geometry>
         <material name="arm_link_wr1">
@@ -426,5 +426,5 @@
           <origin xyz="0.118 0.0 -0.07" rpy="1.57 0 0" />
         <geometry>
-          <mesh filename="file://$(find spot_description)/meshes/arm/collision/left_finger_2.stl" scale="1000 1000 1000"/>
+          <mesh filename="file://$(find spot_description)/meshes/arm/collision/left_finger.stl" scale="1000 1000 1000"/>
         </geometry>
       </collision>
@@ -447,4 +447,8 @@
         <gazebo reference="${tf_prefix}left_finger_link">
             <material>Gazebo/DarkGrey</material>
+            <mu1>1000.0</mu1>
+            <mu2>1000.0</mu2>
+            <minDepth>0.003</minDepth>
+            <maxVel>0</maxVel>
         </gazebo>
         <link name="${tf_prefix}right_finger_link">
@@ -452,5 +456,5 @@
         <origin xyz="0.118 0.02 -0.07" rpy="1.57 0 0" />
         <geometry>
-          <mesh filename="file://$(find spot_description)/meshes/arm/visual/right_finger_2.stl" scale="1000 1000 1000"/>
+          <mesh filename="file://$(find spot_description)/meshes/arm/visual/right_finger.stl" scale="1000 1000 1000"/>
         </geometry>
         <material name="arm_link_wr1">
@@ -461,5 +465,5 @@
           <origin xyz="0.118 0.02 -0.07" rpy="1.57 0 0" />
         <geometry>
-          <mesh filename="file://$(find spot_description)/meshes/arm/collision/right_finger_2.stl" scale="1000 1000 1000"/>
+          <mesh filename="file://$(find spot_description)/meshes/arm/collision/right_finger.stl" scale="1000 1000 1000"/>
         </geometry>
       </collision>
@@ -481,4 +485,8 @@
         <gazebo reference="${tf_prefix}right_finger_link">
             <material>Gazebo/DarkGrey</material>
+            <mu1>1000.0</mu1>
+            <mu2>1000.0</mu2>
+            <minDepth>0.003</minDepth>
+            <maxVel>0</maxVel>
         </gazebo>
         <!-- Extrematies -->
@@ -979,40 +987,4 @@
       <axis xyz="0 0 0"/>
   </joint>
-        <!--gazebo reference="rgb_camera_link_frame">
-            <sensor name="camera" type="wideanglecamera">
-            <camera>
-                <horizontal_fov>6.283</horizontal_fov>
-                    <image>
-                        <width>320</width>
-                        <height>240</height>
-                    </image>
-                    <clip>
-                        <near>0.1</near>
-                        <far>100</far>
-                    </clip>
-                    <lens>
-                        <type>custom</type>
-                        <custom_function>
-                            <c1>1.05</c1>
-                            <c2>4</c2>
-                            <f>1.0</f>
-                            <fun>tan</fun>
-                        </custom_function>
-                        <scale_to_hfov>true</scale_to_hfov>
-                        <cutoff_angle>3.1415</cutoff_angle>
-                        <env_texture_size>512</env_texture_size>
-                    </lens>
-                    <always_on>1</always_on>
-                    <update_rate>30</update_rate>
-            </camera>
-            <plugin name="camera_controller" filename="libgazebo_ros_camera.so">
-                <cameraName>rgb_camera</cameraName>
-                <imageTopicName>image_raw</imageTopicName>
-                <cameraInfoTopicName>camera_info</cameraInfoTopicName>
-                <frameName>rgb_camera_link_frame</frameName>
-                <hackBaseline>0.07</hackBaseline>
-            </plugin>
-            </sensor>
-    </gazebo-->
         <!-- *********************** CAMERA SETUP *********************************  -->
 <!-- Each sensor must be attached to a link.                              -->
@@ -1057,42 +1029,163 @@
         </sensor>
     </gazebo>
-        <!--gazebo reference="camera_link">
-            <sensor name="camera" type="camera">
-                <update_rate>30.0</update_rate>
-                <always_on>1</always_on>
-                <camera name="camera">
-                    <horizontal_fov>1.3962634</horizontal_fov>
-                    <image>
-                        <width>480</width>
-                        <height>360</height>
-                        <format>R8G8B8</format>
-                    </image>
-                    <clip>
-                        <near>0.01</near>
-                        <far>20</far>
-                    </clip>
-                    <distortion>
-                        <k1>0.0</k1>
-                        <k2>0.0</k2>
-                        <k3>0.0</k3>
-                        <p1>0.0</p1>
-                        <p2>0.0</p2>
-                        <center>0.5 0.5</center>
-                    </distortion>
-                </camera>
-                <plugin filename="libgazebo_ros_camera.so" name="camera_controller">
-                    <ros> <namespace>/robot1</namespace>
-                        <remapping>~/image_raw:=camera1/image</remapping>
-                        <remapping>~/camera_info:=camera1/camera_info</remapping>
-                    </ros>
-                    <camera_name>camera_low</camera_name>
-                    <frame_name>camera_link</frame_name>
-                </plugin>
-            </sensor>
-        </gazebo-->
+   <!-- Suction Cup -->
+   <link name="vacuum_gripper">
+      <gravity>0</gravity>
+      <visual>
+        <origin rpy="0 0 0" xyz="0 0 0"/>
+        <geometry>
+          <cylinder radius="0.005" length="0.01"/>
+        </geometry>
+        <material name="transparent">
+          <color rgba="0 0 1 0"/>
+        </material>
+      </visual>
+      <collision>
+        <origin rpy="0 0 0" xyz="0 0 0"/>
+        <geometry>
+          <cylinder radius="0.005" length="0.01"/>
+        </geometry>
+      </collision>
+       <inertial>
+        <origin rpy="0 0 0" xyz="0.000000 0.000000 0.000000"/>
+        <mass value="0.0001"/>
+        <inertia ixx="1e-08" ixy="0" ixz="0" iyy="1e-08" iyz="0" izz="1e-08"/>
+      </inertial>
+    </link>
+    <joint name="gripper_joint" type="revolute">
+      <axis xyz="1 0 0" />
+      <parent link="${tf_prefix}arm_link_wr1" />
+      <child link="vacuum_gripper" />
+      <origin rpy="0 1.5708 0" xyz="0.26 0.0125 0" />
+      <limit effort="50" velocity="50" lower="0" upper="0" />
+      <dynamics damping="0.0" friction="10"/>
+    </joint>
+    <gazebo>
+      <plugin name="gazebo_ros_vacuum_gripper" filename="libgazebo_ros_vacuum_gripper.so">
+        <!--robotNamespace>/spot/vacuum_gripper</robotNamespace-->
+          <link_name>vacuum_gripper</link_name>
+          <!-- Remapping service and topic names -->
+        <remapping>switch:=custom_switch1</remapping>
+        <remapping>grasping:=custom_grasping1</remapping>
+        <bodyName>vacuum_gripper</bodyName>
+        <!--topicName>grasping_vacuum</topicName-->
+          <!--serviceName>toggle</serviceName-->
+	    <maxForce>500</maxForce>
+        <maxDistance>0.05</maxDistance>
+        <minDistance>0.01</minDistance>
+      </plugin>
+  </gazebo>
+     <gazebo reference="vacuum_gripper">
+        <material>Gazebo/Blue</material>
+    </gazebo>
+    <link name="vacuum_gripper2">
+      <gravity>0</gravity>
+      <visual>
+        <origin rpy="0 0 0" xyz="0 0 0"/>
+        <geometry>
+          <cylinder radius="0.005" length="0.01"/>
+        </geometry>
+        <material name="transparent">
+          <color rgba="0 0 1 0"/>
+        </material>
+      </visual>
+      <collision>
+        <origin rpy="0 0 0" xyz="0 0 0"/>
+        <geometry>
+          <cylinder radius="0.005" length="0.01"/>
+        </geometry>
+      </collision>
+        <inertial>
+        <origin rpy="0 0 0" xyz="0.000000 0.000000 0.000000"/>
+        <mass value="0.0001"/>
+        <inertia ixx="1e-08" ixy="0" ixz="0" iyy="1e-08" iyz="0" izz="1e-08"/>
+      </inertial>
+    </link>
+    <joint name="gripper_joint2" type="revolute">
+      <axis xyz="1 0 0" />
+      <parent link="${tf_prefix}arm_link_wr1" />
+      <child link="vacuum_gripper2" />
+      <origin rpy="0 1.5708 0" xyz="0.26 -0.0125 0" />
+      <limit effort="50" velocity="50" lower="0" upper="0" />
+      <dynamics damping="0.0" friction="10"/>
+    </joint>
+    <gazebo reference="vacuum_gripper2">
+        <material>Gazebo/Green</material>
+    </gazebo>
+     <gazebo>
+      <plugin name="gazebo_ros_vacuum_gripper2" filename="libgazebo_ros_vacuum_gripper.so">
+        <robotNamespace>/spot/vacuum_gripper2</robotNamespace>
+          <link_name>vacuum_gripper2</link_name>
+          <!-- Remapping service and topic names -->
+        <remapping>switch:=custom_switch2</remapping>
+        <remapping>grasping:=custom_grasping2</remapping>
+        <bodyName>vacuum_gripper2</bodyName>
+        <!--topicName>grasping_vacuum</topicName-->
+          <!--serviceName>toggle</serviceName-->
+	    <maxForce>500</maxForce>
+        <maxDistance>0.05</maxDistance>
+        <minDistance>0.01</minDistance>
+      </plugin>
+  </gazebo>
+    <link name="vacuum_gripper3">
+      <gravity>0</gravity>
+      <visual>
+        <origin rpy="0 0 0" xyz="0 0 0"/>
+        <geometry>
+          <cylinder radius="0.005" length="0.01"/>
+        </geometry>
+        <material name="transparent">
+          <color rgba="0 0 1 0"/>
+        </material>
+      </visual>
+      <collision>
+        <origin rpy="0 0 0" xyz="0 0 0"/>
+        <geometry>
+          <cylinder radius="0.005" length="0.01"/>
+        </geometry>
+      </collision>
+        <inertial>
+        <origin rpy="0 0 0" xyz="0.000000 0.000000 0.000000"/>
+        <mass value="0.0001"/>
+        <inertia ixx="1e-08" ixy="0" ixz="0" iyy="1e-08" iyz="0" izz="1e-08"/>
+      </inertial>
+    </link>
+    <joint name="gripper_joint3" type="revolute">
+      <axis xyz="1 0 0" />
+      <parent link="${tf_prefix}arm_link_wr1" />
+      <child link="vacuum_gripper3" />
+      <origin rpy="0 1.5708 0" xyz="0.26 0 0.0125" />
+      <limit effort="50" velocity="50" lower="0" upper="0" />
+      <dynamics damping="0.0" friction="10"/>
+    </joint>
+    <gazebo reference="vacuum_gripper3">
+        <material>Gazebo/Red</material>
+    </gazebo>
+     <gazebo>
+      <plugin name="gazebo_ros_vacuum_gripper3" filename="libgazebo_ros_vacuum_gripper.so">
+        <robotNamespace>/spot/vacuum_gripper3</robotNamespace>
+          <link_name>vacuum_gripper3</link_name>
+          <!-- Remapping service and topic names -->
+        <remapping>switch:=custom_switch3</remapping>
+        <remapping>grasping:=custom_grasping3</remapping>
+        <bodyName>vacuum_gripper3</bodyName>
+        <!--topicName>grasping_vacuum</topicName-->
+          <!--serviceName>toggle</serviceName-->
+	    <maxForce>500</maxForce>
+        <maxDistance>0.05</maxDistance>
+        <minDistance>0.01</minDistance>
+      </plugin>
+  </gazebo>
         <!-- Standard accessories. -->
         <!--xacro:include filename="$(find spot_description)/urdf/accessories.urdf.xacro" /-->
         <!-- Optional custom includes. -->
         <!--xacro:include filename="$(optenv SPOT_URDF_EXTRAS empty.urdf)" /-->
+        <!--gazebo>
+            <plugin name="gazebo_ros_vacuum_gripper" filename="libgazebo_ros_vacuum_gripper.so">
+                <robotNamespace>/vacuum_gripper</robotNamespace>
+                <link_name>${tf_prefix}arm_link_fngr</link_name>
+                <topicName>grasping</topicName>
+            </plugin>
+        </gazebo-->
     </xacro:macro>
 </robot>

Commit message: Add 3 suction cups

File: spot_description/urdf/spot_macro_control.xacro (robot description, xacro)
@@ -1155,5 +1155,5 @@
       <parent link="${tf_prefix}arm_link_wr1" />
       <child link="vacuum_gripper3" />
-      <origin rpy="0 1.5708 0" xyz="0.26 0 0.0125" />
+      <origin rpy="0 1.5708 0" xyz="0.26 0  0.0125" />
       <limit effort="50" velocity="50" lower="0" upper="0" />
       <dynamics damping="0.0" friction="10"/>

Commit message: changes to 4 vacuum cups array Create the Link attacher gazebo plugin and inplemented in the spot_empty.world

File: spot_description/urdf/spot_macro_control.xacro (robot description, xacro)
@@ -417,5 +417,5 @@
         <origin xyz="0.118 0.0 -0.07" rpy="1.57 0 0" />
         <geometry>
-          <mesh filename="file://$(find spot_description)/meshes/arm/visual/left_finger.stl" scale="1000 1000 1000"/>
+          <mesh filename="file://$(find spot_description)/meshes/arm/visual/left_finger_3.stl" scale="1000 1000 1000"/>
         </geometry>
         <material name="arm_link_wr1">
@@ -426,5 +426,5 @@
           <origin xyz="0.118 0.0 -0.07" rpy="1.57 0 0" />
         <geometry>
-          <mesh filename="file://$(find spot_description)/meshes/arm/collision/left_finger.stl" scale="1000 1000 1000"/>
+          <mesh filename="file://$(find spot_description)/meshes/arm/collision/left_finger_3.stl" scale="1000 1000 1000"/>
         </geometry>
       </collision>
@@ -456,5 +456,5 @@
         <origin xyz="0.118 0.02 -0.07" rpy="1.57 0 0" />
         <geometry>
-          <mesh filename="file://$(find spot_description)/meshes/arm/visual/right_finger.stl" scale="1000 1000 1000"/>
+          <mesh filename="file://$(find spot_description)/meshes/arm/visual/right_finger_3.stl" scale="1000 1000 1000"/>
         </geometry>
         <material name="arm_link_wr1">
@@ -465,5 +465,5 @@
           <origin xyz="0.118 0.02 -0.07" rpy="1.57 0 0" />
         <geometry>
-          <mesh filename="file://$(find spot_description)/meshes/arm/collision/right_finger.stl" scale="1000 1000 1000"/>
+          <mesh filename="file://$(find spot_description)/meshes/arm/collision/right_finger_3.stl" scale="1000 1000 1000"/>
         </geometry>
       </collision>
@@ -1057,6 +1057,6 @@
       <parent link="${tf_prefix}arm_link_wr1" />
       <child link="vacuum_gripper" />
-      <origin rpy="0 1.5708 0" xyz="0.26 0.0125 0" />
-      <limit effort="50" velocity="50" lower="0" upper="0" />
+      <origin rpy="0 1.5708 0" xyz="0.256 0.0125 -0.015" />
+      <limit effort="500" velocity="50" lower="0" upper="0" />
       <dynamics damping="0.0" friction="10"/>
     </joint>
@@ -1106,6 +1106,6 @@
       <parent link="${tf_prefix}arm_link_wr1" />
       <child link="vacuum_gripper2" />
-      <origin rpy="0 1.5708 0" xyz="0.26 -0.0125 0" />
-      <limit effort="50" velocity="50" lower="0" upper="0" />
+      <origin rpy="0 1.5708 0" xyz="0.256 -0.0125 -0.015" />
+      <limit effort="500" velocity="50" lower="0" upper="0" />
       <dynamics damping="0.0" friction="10"/>
     </joint>
@@ -1155,6 +1155,6 @@
       <parent link="${tf_prefix}arm_link_wr1" />
       <child link="vacuum_gripper3" />
-      <origin rpy="0 1.5708 0" xyz="0.26 0  0.0125" />
-      <limit effort="50" velocity="50" lower="0" upper="0" />
+      <origin rpy="0 1.5708 0" xyz="0.256 -0.0125  0.005" />
+      <limit effort="500" velocity="50" lower="0" upper="0" />
       <dynamics damping="0.0" friction="10"/>
     </joint>
@@ -1162,5 +1162,5 @@
         <material>Gazebo/Red</material>
     </gazebo>
-     <gazebo>
+        <gazebo>
       <plugin name="gazebo_ros_vacuum_gripper3" filename="libgazebo_ros_vacuum_gripper.so">
         <robotNamespace>/spot/vacuum_gripper3</robotNamespace>
@@ -1170,4 +1170,53 @@
         <remapping>grasping:=custom_grasping3</remapping>
         <bodyName>vacuum_gripper3</bodyName>
+        <!--topicName>grasping_vacuum</topicName-->
+          <!--serviceName>toggle</serviceName-->
+	    <maxForce>500</maxForce>
+        <maxDistance>0.05</maxDistance>
+        <minDistance>0.01</minDistance>
+      </plugin>
+  </gazebo>
+    <link name="vacuum_gripper4">
+      <gravity>0</gravity>
+      <visual>
+        <origin rpy="0 0 0" xyz="0 0 0"/>
+        <geometry>
+          <cylinder radius="0.005" length="0.01"/>
+        </geometry>
+        <material name="transparent">
+          <color rgba="0 0 1 0"/>
+        </material>
+      </visual>
+      <collision>
+        <origin rpy="0 0 0" xyz="0 0 0"/>
+        <geometry>
+          <cylinder radius="0.005" length="0.01"/>
+        </geometry>
+      </collision>
+        <inertial>
+        <origin rpy="0 0 0" xyz="0.000000 0.000000 0.000000"/>
+        <mass value="0.0001"/>
+        <inertia ixx="1e-08" ixy="0" ixz="0" iyy="1e-08" iyz="0" izz="1e-08"/>
+      </inertial>
+    </link>
+    <joint name="gripper_joint4" type="revolute">
+      <axis xyz="1 0 0" />
+      <parent link="${tf_prefix}arm_link_wr1" />
+      <child link="vacuum_gripper4" />
+      <origin rpy="0 1.5708 0" xyz="0.256 0.0125  0.005" />
+      <limit effort="500" velocity="50" lower="0" upper="0" />
+      <dynamics damping="0.0" friction="10"/>
+    </joint>
+    <gazebo reference="vacuum_gripper4">
+        <material>Gazebo/Red</material>
+    </gazebo>
+        <gazebo>
+      <plugin name="gazebo_ros_vacuum_gripper4" filename="libgazebo_ros_vacuum_gripper.so">
+        <robotNamespace>/spot/vacuum_gripper4</robotNamespace>
+          <link_name>vacuum_gripper4</link_name>
+          <!-- Remapping service and topic names -->
+        <remapping>switch:=custom_switch4</remapping>
+        <remapping>grasping:=custom_grasping4</remapping>
+        <bodyName>vacuum_gripper4</bodyName>
         <!--topicName>grasping_vacuum</topicName-->
           <!--serviceName>toggle</serviceName-->

Commit message: changes the chip model

File: spot_description/urdf/spot_macro_control.xacro (robot description, xacro)
@@ -1035,5 +1035,5 @@
         <origin rpy="0 0 0" xyz="0 0 0"/>
         <geometry>
-          <cylinder radius="0.005" length="0.01"/>
+          <cylinder radius="0.002" length="0.01"/>
         </geometry>
         <material name="transparent">
@@ -1077,5 +1077,5 @@
   </gazebo>
      <gazebo reference="vacuum_gripper">
-        <material>Gazebo/Blue</material>
+        <material>Gazebo/Grey</material>
     </gazebo>
     <link name="vacuum_gripper2">
@@ -1084,5 +1084,5 @@
         <origin rpy="0 0 0" xyz="0 0 0"/>
         <geometry>
-          <cylinder radius="0.005" length="0.01"/>
+          <cylinder radius="0.002" length="0.01"/>
         </geometry>
         <material name="transparent">
@@ -1111,5 +1111,5 @@
     </joint>
     <gazebo reference="vacuum_gripper2">
-        <material>Gazebo/Green</material>
+        <material>Gazebo/Grey</material>
     </gazebo>
      <gazebo>
@@ -1133,5 +1133,5 @@
         <origin rpy="0 0 0" xyz="0 0 0"/>
         <geometry>
-          <cylinder radius="0.005" length="0.01"/>
+          <cylinder radius="0.002" length="0.01"/>
         </geometry>
         <material name="transparent">
@@ -1160,5 +1160,5 @@
     </joint>
     <gazebo reference="vacuum_gripper3">
-        <material>Gazebo/Red</material>
+        <material>Gazebo/Grey</material>
     </gazebo>
         <gazebo>
@@ -1182,5 +1182,5 @@
         <origin rpy="0 0 0" xyz="0 0 0"/>
         <geometry>
-          <cylinder radius="0.005" length="0.01"/>
+          <cylinder radius="0.002" length="0.01"/>
         </geometry>
         <material name="transparent">
@@ -1209,5 +1209,5 @@
     </joint>
     <gazebo reference="vacuum_gripper4">
-        <material>Gazebo/Red</material>
+        <material>Gazebo/Grey</material>
     </gazebo>
         <gazebo>
