Commit message: Working simulation

File: spot_description/urdf/spot_macro_control.xacro (robot description, xacro)
@@ -462,5 +462,5 @@
         </material>
       </visual>
-      <collision>
+      <collision name="right_finger_collision">
           <origin xyz="0.118 0.02 -0.07" rpy="1.57 0 0" />
         <geometry>
@@ -484,4 +484,114 @@
         </joint>
         <gazebo reference="${tf_prefix}right_finger_link">
+            <material>Gazebo/DarkGrey</material>
+            <mu1>1000.0</mu1>
+            <mu2>1000.0</mu2>
+            <minDepth>0.003</minDepth>
+            <maxVel>0</maxVel>
+            <sensor name="right_finger_contactsensor_sensor" type="contact">
+                <always_on>true</always_on>
+                <contact>
+                    <collision>right_finger_collision</collision>
+                </contact>
+                <plugin name="right_finger_plugin" filename="libgazebo_ros_bumper.so">
+                    <bumperTopicName>right_finger_contact</bumperTopicName>
+                    <frameName>${tf_prefix}right_finger_link</frameName>
+                </plugin>
+            </sensor>
+        </gazebo>
+        <link name="${tf_prefix}right_finger_link_bar">
+            <visual>
+                <origin rpy="0 0 0" xyz="0 0 0"/>
+                <geometry>
+                    <cylinder radius="0.002" length="0.045"/>
+                </geometry>
+                <material name="arm_link_wr1">
+                <color rgba="0.2 0.2 0.2 1" />
+                </material>
+            </visual>
+            <collision>
+                <origin rpy="0 0 0" xyz="0 0 0"/>
+                <geometry>
+                    <cylinder radius="0.002" length="0.045"/>
+                </geometry>
+            </collision>
+            <collision>
+                <origin rpy="0.0 0.0 0" xyz="0.0 -0.004 0"/>
+                <geometry>
+                    <cylinder radius="0.002" length="0.045"/>
+                </geometry>
+            </collision>
+            <collision>
+                <origin rpy="0.0 0.0 0" xyz="0.0 -0.008 0"/>
+                <geometry>
+                    <cylinder radius="0.002" length="0.045"/>
+                </geometry>
+            </collision>
+            <inertial>
+        <origin rpy="0.006393076449033863 0.2928526604761865 -0.022814984050994802"
+          xyz="0.12516802549362183 0.00010137435310753062 -0.013997982256114483" />
+        <mass value="0.785" />
+        <inertia ixx="0.00076741362048185" ixy="0.0" ixz="0.0" iyy="0.0017628124054271809" iyz="0.0"
+          izz="0.0016818105865345951" />
+      </inertial>
+        </link>
+        <joint name="right_finger_joint_bar" type="fixed">
+            <origin xyz="0.277 0.025 0.003" rpy="1.57 0 0" />
+            <axis xyz="0 1 0" />
+            <parent link="${tf_prefix}right_finger_link" />
+            <child link="${tf_prefix}right_finger_link_bar" />
+            <limit effort="1" velocity="10.00" lower="-0.0" upper="0.03" />
+        </joint>
+         <gazebo reference="${tf_prefix}right_finger_link_bar">
+            <material>Gazebo/DarkGrey</material>
+            <mu1>1000.0</mu1>
+            <mu2>1000.0</mu2>
+            <minDepth>0.003</minDepth>
+            <maxVel>0</maxVel>
+        </gazebo>
+        <link name="${tf_prefix}left_finger_link_bar">
+            <visual>
+                <origin rpy="0 0 0" xyz="0 0 0"/>
+                <geometry>
+                    <cylinder radius="0.002" length="0.045"/>
+                </geometry>
+                <material name="arm_link_wr1">
+                <color rgba="0.2 0.2 0.2 1" />
+                </material>
+            </visual>
+            <collision>
+                <origin rpy="0 0 0" xyz="0 0 0"/>
+                <geometry>
+                    <cylinder radius="0.002" length="0.045"/>
+                </geometry>
+            </collision>
+            <collision>
+                <origin rpy="0.0 0.0 0" xyz="0.0 -0.005 0"/>
+                <geometry>
+                    <cylinder radius="0.003" length="0.045"/>
+                </geometry>
+            </collision>
+            <collision>
+                <origin rpy="0.0 0.0 0" xyz="0.0 -0.01 0"/>
+                <geometry>
+                    <cylinder radius="0.004" length="0.045"/>
+                </geometry>
+            </collision>
+            <inertial>
+        <origin rpy="0.006393076449033863 0.2928526604761865 -0.022814984050994802"
+          xyz="0.12516802549362183 0.00010137435310753062 -0.013997982256114483" />
+        <mass value="0.785" />
+        <inertia ixx="0.00076741362048185" ixy="0.0" ixz="0.0" iyy="0.0017628124054271809" iyz="0.0"
+          izz="0.0016818105865345951" />
+      </inertial>
+        </link>
+        <joint name="left_finger_joint_bar" type="fixed">
+            <origin xyz="0.277 -0.025 0.003" rpy="1.57 0 0" />
+            <axis xyz="0 1 0" />
+            <parent link="${tf_prefix}left_finger_link" />
+            <child link="${tf_prefix}left_finger_link_bar" />
+            <limit effort="1" velocity="10.00" lower="-0.0" upper="0.03" />
+        </joint>
+         <gazebo reference="${tf_prefix}left_finger_link_bar">
             <material>Gazebo/DarkGrey</material>
             <mu1>1000.0</mu1>
@@ -959,5 +1069,5 @@
               <type>gaussian</type>
               <mean>0.0</mean>
-              <stddev>0.001</stddev>
+              <stddev>0.00001</stddev>
           </noise>
           </ray>
@@ -1057,5 +1167,5 @@
       <parent link="${tf_prefix}arm_link_wr1" />
       <child link="vacuum_gripper" />
-      <origin rpy="0 1.5708 0" xyz="0.256 0.0125 -0.015" />
+      <origin rpy="0 1.5708 0" xyz="0.272 0.0125 -0.015" />
       <limit effort="500" velocity="50" lower="0" upper="0" />
       <dynamics damping="0.0" friction="10"/>
@@ -1106,5 +1216,5 @@
       <parent link="${tf_prefix}arm_link_wr1" />
       <child link="vacuum_gripper2" />
-      <origin rpy="0 1.5708 0" xyz="0.256 -0.0125 -0.015" />
+      <origin rpy="0 1.5708 0" xyz="0.272 -0.0125 -0.015" />
       <limit effort="500" velocity="50" lower="0" upper="0" />
       <dynamics damping="0.0" friction="10"/>
@@ -1155,5 +1265,5 @@
       <parent link="${tf_prefix}arm_link_wr1" />
       <child link="vacuum_gripper3" />
-      <origin rpy="0 1.5708 0" xyz="0.256 -0.0125  0.005" />
+      <origin rpy="0 1.5708 0" xyz="0.272 -0.0125  0.005" />
       <limit effort="500" velocity="50" lower="0" upper="0" />
       <dynamics damping="0.0" friction="10"/>
@@ -1204,5 +1314,5 @@
       <parent link="${tf_prefix}arm_link_wr1" />
       <child link="vacuum_gripper4" />
-      <origin rpy="0 1.5708 0" xyz="0.256 0.0125  0.005" />
+      <origin rpy="0 1.5708 0" xyz="0.272 0.0125  0.005" />
       <limit effort="500" velocity="50" lower="0" upper="0" />
       <dynamics damping="0.0" friction="10"/>

File: test_bench_description/urdf/Socket.urdf (robot description, URDF)
Before this commit: robot socket, 7 links, 6 joints
Links:
- added link PressureBar_bar, mass 0.785; collision box size=0.015 0.005 0.08; collision cylinder length=0.1 radius=0.002
- added link cover_box, mass 0.01; collision box size=0.04 0.002 0.04
- link PressureBar: mass 32.86 -> 0.2; geometry visual mesh filename=file://$(find test_bench_description)/meshes/PressureBar.stl
- link bracket: geometry collision mesh filename=file://$(find test_bench_description)/meshes/brackets.stl; visual mesh filename=file://$(find test_bench_description)/meshes/brackets.stl
- link socket: mass 32.86 -> 0.1
Joints:
- added joint collision_bar: type fixed, parent PressureBar, child PressureBar_bar, origin xyz=0.045 0.053 0.002 rpy=1.57 0 1.57, axis 0 1 0, limit lower=-0.0 upper=0.03 effort=1 velocity=10.00
- added joint cover_bar_joint: type fixed, parent cover, child cover_box, origin xyz=-0.03 0.002 0.028 rpy=0 0 0, axis 0 1 0, limit lower=-0.0 upper=0.03 effort=1 velocity=10.00
- joint pcb_Lbracket: origin xyz=0.073 0. 0.073 rpy=1.57 3.14 0 -> xyz=0.073 0.003 0.073 rpy=1.57 3.14 0
- joint pressurebar_cover: limit lower=-0.75 upper=0 effort=1000 velocity=0.50 -> lower=-0.05 upper=0.1 effort=1000 velocity=0.50
- joint pressurebar_virtual_Rbracket: limit lower=-2.5 upper=0. effort=1000 velocity=0.50 -> lower=-1.8 upper=-0.05 effort=1000 velocity=0.50
